File: Schematics/clock/clock.kicad_sch (KiCad schematic)
At the start: 25 parts, among them SW1 SW_Push, SW2 SW_Push, U1 74LS04, U2 LM555, U3 74LS32, U4 74LS08, U5 LM555, U6 LM555

Commit message: Updated schematics
Parts:
- added C10, C9: 0.1µF, Capacitor_THT:C_Disc_D4.3mm_W1.9mm_P5.00mm, symbol Device:C
- added C11, C12: 1uf, symbol Device:C_Polarized
- added C13: 0.1uf, symbol Device:C
- added C8: 22uF, symbol Device:C_Polarized
- added D2: 1N914, Diode_THT:D_DO-35_SOD27_P7.62mm_Horizontal, symbol Diode:1N914
- added J2: Power, symbol Connector_Generic:Conn_01x03
- added R10, R14, R22, R23: 10k, symbol Device:R
- added R11: 47k, symbol Device:R
- added R12: 82k, symbol Device:R
- added R13: 1k, symbol Device:R
- added R15, R16, R17, R18, R19, R20, R21: 220, symbol Device:R
- added R9: 10K, symbol Device:R
- added RV2: 10k, symbol Device:R_Potentiometer
- added SW3: Reset, symbol Switch:SW_Push
- added U10: ATmega328-P, Package_DIP:DIP-28_W7.62mm, symbol MCU_Microchip_ATmega:ATmega328-P
- added U12: 5641AS, Display_7Segment:CA56-12SRWA, symbol Display_Character:CC56-12SRWA
- added U7: LM555, Package_SO:SOIC-8_3.9x4.9mm_P1.27mm, symbol Timer:LM555xM
- added U8: 74LS08, symbol 74xx:74LS08
- added U9: 74HC14, symbol 74xx:74HC14
- SW1: value SW_Push -> Step
- SW2: value SW_Push -> Mode
Connections:
- net GND: now also C10.2, C11.2, C13.1, C9.2, D2.2 (A), J2.1 (Pin_1), J2.3 (Pin_3), R12.2, R22.2, R23.2, R9.2, RV2.2, SW3.1, U10.22 (GND), U10.8 (GND), U7.1 (GND), U9.7 (GND)
- net HLT: now also R9.1
- net VCC: now also C10.1, C8.1, C9.1, J2.2 (Pin_2), R10.1, U7.4 (R), U7.8 (VCC), U9.14 (VCC)
- net at R7.1, U1.1, U6.3 (Q): now also U4.4; no longer U4.2
- net at U1.2: now also U4.2; no longer U4.4
- net CLK renamed CLOCK
- net CLOCK: now also R23.1, U10.4 (PD2), U8.11; no longer U4.8
- net ~{CLK} renamed ~{CLOCK}
- new net: R19.2, U12.1 (e)
- new net: R20.2, U12.10 (f)
- new net: R15.2, U12.11 (a)
- new net: U10.26 (PC3), U12.12 (CC1)
- new net: R18.2, U12.2 (d)
- new net: R17.2, U12.4 (c)
- new net: R21.2, U12.5 (g)
- new net: U10.23 (PC0), U12.6 (CC4)
- new net: R16.2, U12.7 (b)
- new net: U10.24 (PC1), U12.8 (CC3)
- new net: U10.25 (PC2), U12.9 (CC2)
- new net: R18.1, U10.16 (PB2)
- new net: C8.2, RV2.1, U7.2 (TR), U7.6 (THR)
- new net: R14.1, U10.1 (~{RESET}/PC6)
- new net: R15.1, U10.13 (PD7)
- new net: R16.1, U10.14 (PB0)
- new net: R17.1, U10.15 (PB1)
- new net: R19.1, U10.17 (PB3)
- new net: R20.1, U10.18 (PB4)
- new net: R21.1, U10.19 (PB5)
- new net: C12.2, D2.1 (K), R12.1, R13.1
- new net: R13.2, U9.3
- new net: C11.1, R11.2, U9.1
- new net: C12.1, U9.2
- new net: U4.8, U8.12
- new net: U7.3 (Q), U8.13
- new net: R10.2, R11.1, SW3.2
- new net +5V: C13.2, R14.2, U10.20 (AVCC), U10.7 (VCC)
- new net RESET: R22.1, U10.5 (PD3), U9.6
- new net ~{RESET}: U9.4, U9.5
Other:
- note added: "CPU Halt"
- note added: "Clock Select"
- note added: "Frame Counter"
- note added: "Manual Clock"
- note added: "Mode Select"
- note added: "Oscillator"
- note added: "Reset Debounce"
- note added: "Startup Delay"
- note added: "TTL Power"
- moved on the sheet: C6, C7, D1, R8, U1D, U1F, U1G, U3A, U3E, U4A, U4B, U4C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

Commit message: Updates
Parts:
- removed C3, C4: 0.01uF, symbol Device:C
- removed C8: 22uF, symbol Device:C_Polarized
- removed U5: LM555, Package_SO:SOIC-8_3.9x4.9mm_P1.27mm, symbol Timer:LM555xM
- added C1, C2: 1uf, symbol Device:C_Polarized
- added C10: 0.1µF, Capacitor_THT:C_Disc_D4.3mm_W1.9mm_P5.00mm, symbol Device:C
- added C6: 100uF, symbol Device:C_Polarized
- added D1: 1N914, Diode_THT:D_DO-35_SOD27_P7.62mm_Horizontal, symbol Diode:1N914
- added D4: LED, symbol Device:LED
- added J2: Interface, symbol Connector_Generic:Conn_01x08
- added J3: Control, symbol Connector_Generic:Conn_01x04
- added R12, R5: 1k, symbol Device:R
- added R27: 220, symbol Device:R
- added R9: 82k, symbol Device:R
- added unit 6 of U1
- added unit 4 of U1
- added unit 5 of U1
- added U8: 74LS08, symbol 74xx:74LS08
- R3: value 1K -> 10k
- R4: value 1M -> 47k
- renumbered C6 to C11, C7 to C12, C9 to C13, C10 to C14, C5 to C3, C1 to C4, C2 to C5, C12 to C7, C11 to C8, C13 to C9, D1 to D2, D2 to D3, J2 to J1, R9 to R10, R8 to R11, R10 to R13, R11 to R14, R13 to R15, R12 to R16, R15 to R17, R16 to R18, R17 to R19, R5 to R2, R18 to R20, R19 to R21, R20 to R22, R21 to R23, R14 to R24, R23 to R25, R22 to R26, R7 to R6, R2 to R7, R6 to R8, U9 to U1, U6 to U3, U1 to U4, U4 to U5, U8 to U5, U3 to U6, U12 to U9
Connections:
- net CLOCK: now also J2.4 (Pin_4)
- net GND: now also C10.2, C2.2, D1.2 (A), J2.8 (Pin_8), R12.2, R27.1, R9.2, U8.7 (GND); no longer RV2.2
- net RESET: now also J2.6 (Pin_6), U8.3; no longer U1.6
- net VCC: now also C10.1, C6.1, D4.2 (A), J2.1 (Pin_1), U8.14 (VCC); no longer R4.1
- net ~HALT: now reaches U4.8, U5.10
- net MODE_SW_B: now reaches R2.2, R8.1, SW2.1, U3.2 (TR), U3.6 (THR)
- net MODE_SW_B: now also J3.4 (Pin_4)
- net at RV2.1, U7.2 (TR), U7.6 (THR): now also C6.2
- net STEP_SW: now reaches R3.2, SW1.2
- net STEP_SW: now also R4.1, J3.1 (Pin_1)
- net STEP: now reaches U5.5
- net STEP: now also U1.12
- net at R4.2: now also C2.1, U1.9
- net MODE_SW_A: now reaches C3.1, R6.2, SW2.2
- net MODE_SW_A: now also J3.3 (Pin_3)
- net MODE: now reaches R6.1, U3.3 (Q), U4.1, U5.4
- net START_DELAY: now reaches U5.13, U7.3 (Q)
- net START_DELAY: now also J2.2 (Pin_2), U8.2, U8.4
- net RESET_SW: now reaches R13.2, R14.1, SW3.2
- net RESET_SW: now also J3.2 (Pin_2)
- net OSC: now reaches U2.3 (Q), U5.1
- net HLT renamed HALT
- net HALT: now also J2.3 (Pin_3)
- net ~{CLOCK} renamed ~CLOCK
- net ~CLOCK: now also J2.5 (Pin_5)
- net ~{RESET}: no longer names the net of U1.4, U1.5
- net ~{RESET}: now also U8.5
- new net: R12.1, RV2.2
- new net: D4.1 (K), R27.2
- new net: U1.10, U1.13
- new net: C1.2, D1.1 (K), R5.1, R9.1
- new net: U1.6, U8.1
- new net: C1.1, U1.8
- new net: R5.2, U1.11
- new net ~RESET: J2.7 (Pin_7), U8.6
Other:
- note added: "(+)"
- note added: "(-)"
- note added: "Headers"
- note added: "Power"
- note removed: "TTL Power"
- moved on the sheet: C11, C12, C13, C14, C3, C7, C8, C9, D2, D3, J1, R10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
