File: Projects/Clock Module/schematic/clock.kicad_sch (KiCad schematic)
At the start: 63 parts, among them J1 Power, J2 Interface, J3 Control, SW1 Step, SW2 Mode, SW3 Reset, U1 74HC14, U10 ATmega328-P, U2 LM555, U3 LM555, U4 74LS04, U5 74LS08, U6 74LS32, U7 LM555, U8 74LS08, U9 5641AS

Commit message: Built the framework for the emulator, and added a new clock module using JK Flip-Flops
Other:
- added sheet SelectorPanel (untitled.kicad_sch)
Changed lines of the file:
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@@
+    )
+  )
+  (sheet (at 388.62 227.33) (size 12.7 8.89) (fields_autoplaced)
+    (stroke (width 0.1524) (type solid))
+    (fill (color 0 0 0 0.0000))
+    (property "Sheetname" "SelectorPanel" (at 388.62 226.6184 0)
+      (effects (font (size 1.27 1.27)) (justify left bottom))
+    )
+    (property "Sheetfile" "untitled.kicad_sch" (at 388.62 236.8046 0)
+      (effects (font (size 1.27 1.27)) (justify left top))
+    )
+    (instances
+      (project "clock"
+        (path "/2443a44d-7077-4f22-9dfe-ab8f8af6a93f" (page "2"))
+      )
     )
   )

Commit message: Updated clock to use the selector panel
Parts:
- removed C3: 1uF, symbol Device:C_Polarized
- removed J3: Control, symbol Connector_Generic:Conn_01x04
- removed R10, R2, R8: 10K, symbol Device:R
- removed R6: 100K, symbol Device:R
- removed SW2: Mode, symbol Switch:SW_Push
- removed U3: LM555, Package_SO:SOIC-8_3.9x4.9mm_P1.27mm, symbol Timer:LM555xM
- removed unit 7 of U4
- removed unit 1 of U4
- removed unit 6 of U4
- added C10, C11, C9: 0.1µF, Capacitor_THT:C_Disc_D4.3mm_W1.9mm_P5.00mm, symbol Device:C
- added D3, D5, D6, D8: LED, symbol Device:LED
- added R22, R25, R27, R30: 220, symbol Device:R
- added R24, R26, R29: 680, symbol Device:R
- added SW3: SW_Manual, symbol Switch:SW_Push
- added SW4: SW_Slow, symbol Switch:SW_Push
- added SW5: SW_Fast, symbol Switch:SW_Push
- added unit 6 of U10
- added unit 3 of U10
- added unit 2 of U10
- added unit 4 of U10
- added unit 7 of U10
- added unit 5 of U10
- added U11, U13: 74LS73, symbol 74xx:74LS73
- added U12: 74LS32, symbol 74xx:74LS32
- added unit 2 of U7
- added unit 3 of U7
- added unit 4 of U7
- added U8: 74LS93, symbol 74xx:74LS93
- added unit 3 of U9
- added unit 4 of U9
- added X1: SG-7050CCN, Oscillator:Oscillator_SMD_SeikoEpson_SG8002CA-4Pin_7.0x5.0mm, symbol Oscillator:SG-7050CCN
- J1: renamed from J2; value Interface -> Clock Interface
- renumbered C6 to C1, C10 to C13, C11 to C14, C13 to C15, C14 to C16, C9 to C2, C1 to C3, C2 to C4, C4 to C5, C5 to C6, D3 to D4, D4 to D7, J1 to J2, R9 to R10, R21 to R11, R22 to R12, R23 to R13, R12 to R14, R24 to R15, R25 to R16, R26 to R17, R11 to R18, R13 to R19, R3 to R2, R14 to R20, R15 to R21, R16 to R23, R27 to R28, R17 to R3, R18 to R6, R19 to R7, R7 to R8, R20 to R9, SW3 to SW2, U4 to U10, U7 to U2, U2 to U3, U9 to U4, U10 to U5, U5 to U6, U6 to U7, U8 to U9
Connections:
- net +5V: now also C1.1, C12.1, C13.1, C14.1, C15.1, C16.1, D7.2 (A), J2.1 (Pin_1), J2.3 (Pin_3), R1.1, R19.1, R2.1, U1.14 (VCC), U2.4 (R), U2.8 (VCC), U3.4 (R), U3.8 (VCC), U6.14 (VCC), U7.14 (VCC), U9.14 (VCC), C10.1, C11.1, C9.1, SW3.2, SW4.2, SW5.2, U10.14 (VCC), U11.2 (~{R}), U11.4 (VCC), U11.6 (~{R}), U12.14 (VCC), U13.2 (~{R}), U13.4 (VCC), U13.6 (~{R}), U8.5 (VCC), X1.1 (OE), X1.4 (Vcc)
- net CLOCK: now also J1.3 (Pin_3), U8.14 (CP0); no longer J1.4 (Pin_4)
- net GND: now also J2.2 (Pin_2), C10.2, C11.2, C9.2, R22.2, R24.2, R25.2, R26.2, R27.2, R29.2, R30.2, U10.7 (GND), U11.11 (GND), U12.12, U12.13, U12.7 (GND), U13.11 (GND), U7.10, U7.12, U7.13, U7.9, U8.10 (GND), U8.2 (R0(1)), U8.3 (R0(2)), U9.10, U9.12, U9.13, U9.9, X1.2 (GND); no longer J1.8 (Pin_8), J2.1 (Pin_1), J2.3 (Pin_3)
- net HALT: now also J1.2 (Pin_2), U10.1; no longer J1.3 (Pin_3), U10.9
- net RESET: now also J1.8 (Pin_8), U10.3, U11.7 (J), U12.1; no longer J1.6 (Pin_6)
- net START_DELAY: now also J1.1 (Pin_1); no longer J1.2 (Pin_2), U9.4
- net STEP: now also U9.4; no longer U6.5
- net at U7.3: now also U7.4; no longer U6.9
- net at U1.4, U1.5: no longer U9.5
- net MODE_SLOW: now reaches U6.2
- net MODE_SLOW: now also D6.2 (A), U13.9 (Q)
- net MODE renamed FAST_OSC
- net FAST_OSC: now also X1.3 (OUT)
- net OSC renamed SLOW_OSC
- net STEP_SW: no longer names the net of R2.2, R4.1, SW1.2
- removed net VCC: C1.1, C12.1, C13.1, C14.1, C15.1, C16.1, D7.2 (A), J1.1 (Pin_1), J2.2 (Pin_2), R1.1, R19.1, R2.1, U1.14 (VCC), U2.4 (R), U2.8 (VCC), U3.4 (R), U3.8 (VCC), U6.14 (VCC), U7.14 (VCC), U9.14 (VCC)
- net ~CLOCK renamed PHI_4
- net PHI_4: now also U8.9 (Q1)
- net ~HALT: no longer names the net of U6.10
- net ~HALT: now also U10.2; no longer U10.8
- net ~RESET: no longer names the net of U9.6
- net ~RESET: now also U7.5; no longer J1.7 (Pin_7)
- new net: D6.1 (K), R27.1
- new net: U10.12, U13.3 (K)
- new net: R29.1, SW5.1, U10.13, U12.10, U13.14 (J)
- new net: R24.1, SW3.1, U10.5, U11.14 (J), U12.2
- new net: U10.6, U11.3 (K)
- new net: U10.10, U13.10 (K)
- new net: U10.8, U11.1 (C), U11.5 (C), U13.1 (C), U13.5 (C)
- new net: R26.1, SW4.1, U10.11, U12.9, U13.7 (J)
- new net: U12.5, U12.8
- new net: D5.1 (K), R25.1
- new net: D8.1 (K), R30.1
- new net: U10.4, U11.10 (K)
- new net: D3.1 (K), R22.1
- new net: U6.9, U7.6
- new net: U10.9, U12.6
- new net: U12.3, U12.4
- new net MODE_FAST: D8.2 (A), U13.12 (Q), U6.5
- new net MODE_RESET: D3.2 (A), U11.9 (Q)
- new net MODE_STEP: D5.2 (A), U11.12 (Q), U9.5
- new net PHI_16: J1.7 (Pin_7), U8.11 (Q3)
- new net PHI_2: J1.4 (Pin_4), U8.1 (CP1..3), U8.12 (Q0)
- new net PHI_8: J1.6 (Pin_6), U8.8 (Q2)
- no-connect marks 3 -> 24
Other:
- removed sheet SelectorPanel
- note added: "Frequency Divider"
- note added: "Slow Oscillator"
- note added: "try putting a buffer here to reduce the resistor value"
- note removed: "CPU Halt"
- note removed: "Mode Select"
- moved on the sheet: C1, C13, C14, C15, C16, C2, C3, C4, C5, C6, C7, C8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

Commit message: Updated clock
Parts:
- added C17: 0.1µF, Capacitor_THT:C_Disc_D4.3mm_W1.9mm_P5.00mm, symbol Device:C
- added R31: 10k, symbol Device:R
- R24, R26, R29: value 680 -> 1k
Connections:
- net +5V: now also R31.2; no longer U11.2 (~{R}), U11.6 (~{R}), U13.2 (~{R}), U13.6 (~{R})
- net GND: now also C17.1
- net RESET_SW: no longer names the net of R19.2, R20.1, SW2.2
- new net: C17.2, R31.1, U11.2 (~{R}), U11.6 (~{R}), U13.2 (~{R}), U13.6 (~{R})
Other:
- note added: "74HC14 debounce"
- note added: "put another switch in here to stop (disable all modes)"
- note added: "replace with STEP"
- note removed: "try putting a buffer here to reduce the resistor value"
- moved on the sheet: D3, D5, D6, D8, R19, R2, R22, R25, R27, R30

Commit message: Updated the clock circuit
Parts:
- removed C1: 100uF, symbol Device:C_Polarized
- removed RV2: 10k, symbol Device:R_Potentiometer
- removed SW3: SW_Manual, symbol Switch:SW_Push
- removed U2: LM555, Package_SO:SOIC-8_3.9x4.9mm_P1.27mm, symbol Timer:LM555xM
- removed unit 4 of U6
- removed unit 3 of U9
- removed unit 1 of U9
- removed unit 4 of U9
- added D10, D9: LED, symbol Device:LED
- added R32: 220, symbol Device:R
- added SW6: Stop, symbol Switch:SW_Push
- C6: value 1uF -> 22uF
- R14: value 1k -> 220
- R24: value 1k -> 10k
- RV1: value 1M -> 100k
- renumbered U9 to U6
Connections:
- net START_DELAY is gone; now on net HALT: J1.1 (Pin_1)
- net CLOCK: now also J1.2 (Pin_2), U6.11; no longer J1.3 (Pin_3)
- net GND: now also R14.1, R32.2, SW6.1; no longer R14.2
- net HALT: now also R24.1, D9.2 (A); no longer J1.2 (Pin_2)
- net MODE_STEP: now also U6.10; no longer U6.5
- net PHI_16: now also J1.6 (Pin_6); no longer J1.7 (Pin_7)
- net PHI_2: now also J1.3 (Pin_3); no longer J1.4 (Pin_4)
- net PHI_4: now also J1.4 (Pin_4); no longer J1.5 (Pin_5)
- net PHI_8: now also J1.5 (Pin_5); no longer J1.6 (Pin_6)
- net RESET: now also J1.7 (Pin_7), U1.6, D10.2 (A); no longer J1.8 (Pin_8)
- net STEP: now also U10.5, U11.14 (J), U12.2, U6.9; no longer U6.4
- net at U10.2: now also U6.13; no longer U6.10
- net at C17.2, R31.1, U11.2 (~{R})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: now also SW6.2
- net at U7.6: now also U6.12; no longer U6.9
- net at U7.5: now also U6.8; no longer U6.6
- net ~RESET: now reaches U1.4, U1.5
- net ~RESET: now also J1.8 (Pin_8)
- new net: D10.1 (K), R32.1
- new net: D9.1 (K), R14.2
- no-connect marks 24 -> 19
Other:
- note removed: "Startup Delay"
- note removed: "put another switch in here to stop (disable all modes)"
- note removed: "replace with STEP"
- moved on the sheet: C10, C11, C12, C13, C14, C15, C16, C17, C2, C3, C4, C7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
